File: DEMO_touch_MPR121_circuit/DEMO_touch_MPR121_circuit.sch (KiCad schematic (older format))
At the start: 12 parts, among them J1 Conn_01x10_Male, Q1 IPP060N06N, Q2 IPP060N06N, Q3 IPP060N06N

Commit message: circuit schematics updated, new purchase order logged
Parts:
- added 1: ARDUINO_R3_ICSP, symbol Adafruit_MPR121_Capacitive_Touch_Shield-eagle-import:ARDUINO_R3_ICSP
- added 2: MPR121_Arduino_shield, symbol Adafruit_MPR121_Capacitive_Touch_Shield-eagle-import:MPR121_Arduino_shield
- added JP1: HEADER-1X10, symbol Adafruit_MPR121_Capacitive_Touch_Shield-eagle-import:HEADER-1X10
- added U1: VREG_board_MAKERFACTORY, symbol Adafruit_MPR121_Capacitive_Touch_Shield-eagle-import:VREG_board_MAKERFACTORY
Connections:
- net labels added: +5V, 21-7*2.8=1.4V, 3V, 5V, ARDUINO_PROTOSHIELD_BARE_PCB, AREF, Arduino_supply, D13, Headers_to_DEMO_board, LED_array, LED_drive, LED_ring, LED_row1, LED_row2, SCL, SDA, Sparkfun_Dev-13819, VIN, Voltage_stepup
- net labels removed: 21-7.28=1.4V, GNDPWR, black, blue
- wire segments 36 -> 89
- no-connect marks 0 -> 3
Other:
- moved on the sheet: J1, Q1, Q2, Q3, R1, R2, R3, R4, R5, R6, R7, R8

Commit message: circuit schematics reviewed, BOM created ().xlsx)
Parts:
- renumbered 1 to U1, 2 to U2, U1 to U4
Connections:
- net labels added: D2
- wire segments 89 -> 94
- no-connect marks 3 -> 73
Changed lines of the file:
@@
 $EndComp
 $Comp
-L Adafruit_MPR121_Capacitive_Touch_Shield-eagle-import:ARDUINO_R3_ICSP 1
+L Adafruit_MPR121_Capacitive_Touch_Shield-eagle-import:ARDUINO_R3_ICSP U1
 U 1 1 5FB5395C
 P 2300 5750
-F 0 "1" H 2350 5800 118 0001 C CNN
+F 0 "U1" H 2350 5800 118 0001 C CNN
 F 1 "ARDUINO_R3_ICSP" H 2300 5750 118 0001 C CNN
 F 2 "" H 2300 5750 118 0001 C CNN
-F 3 "" H 2300 5750 118 0001 C CNN
+F 3 "https://store.arduino.cc/arduino-uno-rev3" H 2300 5750 118 0001 C CNN
 	1    2300 5750
 	1    0    0    -1
@@
 +5V
 $Comp
-L Adafruit_MPR121_Capacitive_Touch_Shield-eagle-import:MPR121_Arduino_shield 2
+L Adafruit_MPR121_Capacitive_Touch_Shield-eagle-import:MPR121_Arduino_shield U2
 U 1 1 5FB78377
 P 6650 5750
-F 0 "2" H 6700 5800 118 0001 C CNN
+F 0 "U2" H 6700 5800 118 0001 C CNN
 F 1 "MPR121_Arduino_shield" H 7900 5900 118 0001 C CNN
 F 2 "" H 6650 5750 118 0001 C CNN
-F 3 "" H 6650 5750 118 0001 C CNN
+F 3 "https://www.adafruit.com/product/2024" H 6650 5750 118 0001 C CNN
 	1    6650 5750
 	1    0    0    -1
@@
 	3600 5950 3650 5950
 $Comp
-L Adafruit_MPR121_Capacitive_Touch_Shield-eagle-import:VREG_board_MAKERFACTORY U1
+L Adafruit_MPR121_Capacitive_Touch_Shield-eagle-import:VREG_board_MAKERFACTORY U4
 U 1 1 5FB9DFE2
 P 8850 1950
-F 0 "U1" H 8850 2297 42  0000 C CNN
+F 0 "U4" H 8850 2297 42  0001 C CNN
 F 1 "VREG_board_MAKERFACTORY" H 8850 2218 42  0000 C CNN
 F 2 "" H 8850 1950 118 0001 C CNN
-F 3 "" H 8850 1950 118 0001 C CNN
+F 3 "https://asset.conrad.com/media10/add/160267/c1/-/gl/002134132ML00/mode-demploi-2134132-makerfactory-mf-6402396-1-pcs.pdf" H 8850 1950 118 0001 C CNN
 	1    8850 1950
 	1    0    0    -1
@@
 Text Label 3850 1400 1    50   ~ 0
 5V
-NoConn ~ 3850 1050
 Wire Wire Line
 	3850 1400 3850 1150
 Text Label 3750 1400 1    50   ~ 0
 3V
-NoConn ~ 3750 1050
 Wire Wire Line
 	3750 1400 3750 1150
@@
 Wire Wire Line
 	8300 2050 8450 2050
-NoConn ~ 9300 1850
 Wire Wire Line
 	9250 2050 9400 2050
@@
 Text Label 800  2000 0    50   ~ 0
 LED_ring
+Text GLabel 8550 3000 1    50   Input ~ 0
+D2
+Text GLabel 4200 3450 1    50   Input ~ 0
+D2
+Wire Wire Line
+	4200 3550 4200 3450
+NoConn ~ 9250 1850
+NoConn ~ 6850 3550
+NoConn ~ 7150 3550
+NoConn ~ 7350 3550
+NoConn ~ 7450 3550
+NoConn ~ 7550 3550
+NoConn ~ 7750 3550
+NoConn ~ 7850 3550
+NoConn ~ 8050 3550
+NoConn ~ 8250 3550
+NoConn ~ 8350 3550
+NoConn ~ 8650 3550
+NoConn ~ 8750 3550
+NoConn ~ 8850 5950
+NoConn ~ 8750 5950
+NoConn ~ 8650 5950
+NoConn ~ 8550 5950
+NoConn ~ 8450 5950
+NoConn ~ 8350 5950
+NoConn ~ 7750 5950
+NoConn ~ 7650 5950
+NoConn ~ 7550 5950
+NoConn ~ 7450 5950
+NoConn ~ 8000 5050
+NoConn ~ 8000 4900
+NoConn ~ 8000 4750
+NoConn ~ 8850 4750
+NoConn ~ 8850 4900
+NoConn ~ 9900 4650
+NoConn ~ 9900 4550
+NoConn ~ 9900 4750
+NoConn ~ 9900 4850
+NoConn ~ 9900 4950
+NoConn ~ 9900 5050
+NoConn ~ 7100 5050
+NoConn ~ 7100 4900
+NoConn ~ 7100 4750
+NoConn ~ 8200 4450
+NoConn ~ 8200 4250
+NoConn ~ 8600 4550
+NoConn ~ 8600 4350
+NoConn ~ 8600 4150
+NoConn ~ 8200 4050
+NoConn ~ 2800 3550
+NoConn ~ 3000 3550
+NoConn ~ 3100 3550
+NoConn ~ 3200 3550
+NoConn ~ 3400 3550
+NoConn ~ 3500 3550
+NoConn ~ 3700 3550
+NoConn ~ 3900 3550
+NoConn ~ 4000 3550
+NoConn ~ 4300 3550
+NoConn ~ 4400 3550
+NoConn ~ 3200 5950
+NoConn ~ 3300 5950
+NoConn ~ 3400 5950
+NoConn ~ 4000 5950
+NoConn ~ 4100 5950
+NoConn ~ 4200 5950
+NoConn ~ 4300 5950
+NoConn ~ 4400 5950
+NoConn ~ 4500 5950
+NoConn ~ 4550 3100
+NoConn ~ 4750 3100
+NoConn ~ 3750 1150
+NoConn ~ 3850 1150
+NoConn ~ 4300 4450
+NoConn ~ 4300 4650
+NoConn ~ 4300 4850
+NoConn ~ 4700 4950
+NoConn ~ 4700 4750
+NoConn ~ 4700 4550
+Wire Wire Line
+	8550 3550 8550 3100
+Wire Wire Line
+	6750 3550 6750 3100
+Wire Wire Line
+	6750 3100 8550 3100
+Connection ~ 8550 3100
+Wire Wire Line
+	8550 3100 8550 3000
 $EndSCHEMATC
